Commit message: update codebase

File: assets/bundlesdf_napkin_mesh.urdf (robot description, URDF)
Before this commit: robot cube, 1 links, 0 joints
Links:
- link body: mass 0.37 -> 0.056; geometry collision mesh filename=napkin_textured_mesh_with_normals.obj; visual mesh filename=napkin_textured_mesh_with_normals.obj
