Commit message: fix custom cube mesh error

File: assets/bundlesdf_cube_mesh.urdf (robot description, URDF)
Before this commit: robot cube, 1 links, 0 joints
Links:
- link body: geometry collision mesh filename=cube_convex_hull_with_normals.obj; visual mesh filename=cube_convex_hull_with_normals.obj

Commit message: try to fix the trajectory bug

File: assets/bundlesdf_cube_mesh.urdf (robot description, URDF)
Before this commit: robot cube, 1 links, 0 joints
Links:
- link body: geometry collision mesh filename=contactnets_cube.obj; visual mesh filename=contactnets_cube.obj

Commit message: add pretrain arg

File: assets/bundlesdf_cube_mesh.urdf (robot description, URDF)
Before this commit: robot cube, 1 links, 0 joints
Links:
- link body: geometry collision mesh filename=post_processed_mesh_icnn.obj; visual mesh filename=post_processed_mesh_icnn.obj
