Commit message: Correct inertial properties of Franka URDF

File: assets/franka_with_ee.urdf (robot description, URDF)
Before this commit: robot panda, 11 links, 10 joints
Links:
- added link worldfixed
Joints:
- added joint fixed_franka: type fixed, parent worldfixed, child panda_link0, origin xyz=0 0 0.0087 rpy=0 0 0
