Commit message: Update cube URDF to match hand-calculated 'ground-truth' values

File: assets/contactnets_cube.urdf (robot description, URDF)
Before this commit: robot cube, 2 links, 1 joints
Links:
- removed link cube_body
- removed link worldfixed
- added link body, mass 0.37; collision box size=0.1048 0.1048 0.1048; visual box size=0.1048 0.1048 0.1048
Joints:
- removed joint worldfixed_to_cube_body
